File: wvr_v.1.0/wvr_v.1.0.kicad_sch (KiCad schematic)
At the start: 48 parts, among them J1 10118192-0001LF, J2 Conn_01x11, J3 Conn_01x11, SW1 SW_Push, U1 TCMT1101, U2 LM1117-3.3, U3 KLM8G1GETF, U4 PCM5102, U5 ESP32-WROVER-B_(16MB), U6 SeeeduinoXIAO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

Commit message: v3.0
Parts:
- removed U7-C379350: TPS7A0533PDBV, Package_TO_SOT_SMD:SOT-23-5, symbol Regulator_Linear:TPS7A0533PDBV
- added U7: LP5907MFX-1.2, Package_SON:Texas_X2SON-4_1x1mm_P0.65mm, symbol Regulator_Linear:TPS7A05_X2SON
- R13: value 100R -> 1k
- R14: value 1K -> 270R; footprint Resistor_SMD:R_0603_1608Metric_Pad1.05x0.95mm_HandSolder -> Resistor_SMD:R_0402_1005Metric
- R2: value 300 -> 270R
Connections:
- net +3.3VA: now also C17.1, U7.1 (OUT); no longer U4.20 (DVDD)
- net +3V3: now also U4.20 (DVDD)
- net +5V: now also U7.3 (EN), U7.4 (IN)
- net GND: now also U7.2 (GND)
