File: wvr_v.1.0/wvr_v.1.0.kicad_pcb (KiCad board)
At the start: 2 copper layers, 26.6 x 47.7 mm, 44 parts, among them J1 10118192-0001LF, J2 Conn_01x11, J3 Conn_01x11, SW1 SW_Push, U1 TCMT1101, U2 LM1117-3.3, U3 KLM8G1GETF, U4 PCM5102, U5 ESP32-WROVER-B_(16MB)

Commit message: update
Parts:
- removed G***: LOGO, WVR_Maker:WVR_LOGO
- added R14: 1K, Resistor_SMD:R_0603_1608Metric_Pad1.05x0.95mm_HandSolder, B.Cu at (139.7, 35.0)
- added U6: SeeeduinoXIAO, Seeeduino XIAO KICAD:Seeeduino XIAO-MOUDLE14P-2.54-21X17.8MM, B.Cu at (134.6, 44.2)
- R13: value 22 -> 100R
- R2: value 10k -> 300
- SW1: footprint wvr_v.1.0:SW_Push_SPST_NO_Alps_SKRK -> Button_Switch_SMD:SW_Push_SPST_NO_Alps_SKRK
- renumbered B to TP1
Routing:
- net GND: track 104.9 -> 88.5 mm, vias 66 -> 65
- net esp_GPIO21: track 15.2 -> 31.3 mm
- net Net-(R14-Pad2): track 0.00 -> 13.5 mm
- net +5V: track 30.0 -> 40.2 mm, vias 3 -> 2
- net +3V3: track 157.1 -> 164.8 mm, vias 8 -> 9
- net Net-(C6-Pad1): track 7.07 -> 11.2 mm
- net midi_REF: track 10.2 -> 8.02 mm, vias 2 -> 1
- net emmc_CLK: track 24.4 -> 22.9 mm
- net audio_R: track 19.7 -> 18.2 mm, vias 3 -> 1
- net midi_IN: track 19.6 -> 21.0 mm
- net dac_DIN: track 47.4 -> 46.1 mm
- net dac_LRCK: track 42.2 -> 43.1 mm
- net Net-(R10-Pad1): track 5.88 -> 5.05 mm
- net Net-(U6-Pad11): track 0.00 -> 0.76 mm

Commit message: update silk layer, clean up .cpl file, print gerbers
Parts:
- R14: value 1K -> 330; footprint Resistor_SMD:R_0603_1608Metric_Pad1.05x0.95mm_HandSolder -> Resistor_SMD:R_0402_1005Metric; moved to F.Cu
- moved R14 12.2 mm to (131.9, 25.7)
- moved R12 0.75 mm to (131.9, 24.7)
- moved C13 0.22 mm to (131.9, 23.7)
- renumbered TP1 to boot
Routing:
- net Net-(R14-Pad2): track 13.5 -> 42.1 mm, vias 0 -> 1
- net esp_GPIO21: track 31.3 -> 39.5 mm, vias 1 -> 2
- net +3V3: track 164.8 -> 165.8 mm, vias 9 -> 10
- net esp_EN: track 28.1 -> 27.3 mm
- net Net-(C13-Pad2): track 3.20 -> 2.67 mm
- net GND: track 88.5 -> 88.0 mm, vias 65 -> 70
Other:
- board text added: "V 2.1"
- board text removed: "V 1.1"

Commit message: ?
Routing:
- net GND: track 88.0 -> 91.3 mm
- net midi_REF: track 8.02 -> 5.15 mm, vias 1 -> 0
Other:
- board text added: "<———"
- board text added: "D12.A6.T2"
- board text added: "D13.A7.T3"
- board text added: "D6.A0.T0"
- board text added: "MIDI.RX"
- board text added: "MIDI.V+"
- board text added: "WVR V2.1"
- board text removed: "** D13 A7 T3"
- board text removed: "D12 A6 T2"
- board text removed: "D6 A0 T0 **"
- board text removed: "MIDI RX"
- board text removed: "MIDI VREF"
- board text removed: "V 2.1"

Commit message: update IP Address on silk, update jlc component codes
Other:
- board text added: "192.168.4.1"
- board text removed: "192.168.5.18"
Changed lines of the file:
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@@
     (44 Edge.Cuts user hide)
     (45 Margin user hide)
-    (46 B.CrtYd user)
-    (47 F.CrtYd user)
+    (46 B.CrtYd user hide)
+    (47 F.CrtYd user hide)
     (48 B.Fab user hide)
-    (49 F.Fab user)
+    (49 F.Fab user hide)
   )
   (setup
@@
     (effects (font (size 1 1) (thickness 0.153)) (justify mirror))
   )
-  (gr_text 192.168.5.18 (at 144.1 19.08) (layer B.SilkS)
+  (gr_text 192.168.4.1 (at 144.1 19.08) (layer B.SilkS)
     (effects (font (size 2 2) (thickness 0.153)) (justify mirror))
   )
